File: pcb/controller/kicad/expansion-source/service.kicad_sch (KiCad schematic)
At the start: 3 parts, among them J2 43045-0200

Commit message: Simplify mains connectors and separate the 5 V service input
Parts:
- J2: value 43045-0200 -> S2B-XH-A; MPN 43045-0200 -> S2B-XH-A
Changed lines of the file:
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@@
 			)
 		)
-		(property "Value" "43045-0200"
+		(property "Value" "S2B-XH-A"
 			(at 87.3007 109.7936 0)
 			(show_name no)
@@
 			)
 		)
-		(property "Datasheet" "https://www.molex.com/content/dam/molex/molex-dot-com/products/automated/en-us/salesdrawingpdf/430/43045/430450200_sd.pdf"
+		(property "Datasheet" "https://www.jst.com/wp-content/uploads/2025/06/eXH.pdf"
 			(at 101.6 105.41 0)
 			(hide yes)
@@
 			)
 		)
-		(property "MPN" "43045-0200"
+		(property "MPN" "S2B-XH-A"
 			(at 101.6 105.41 0)
 			(hide yes)
